Commit message: Final touches

File: tf_pkg/urdf/robot.urdf (robot description, URDF)
Before this commit: robot foxbot, 2 links, 1 joints
Links:
- added link arm_base_link; collision box size=0.15 0.1 0.1; visual box size=0.15 0.1 0.1
Joints:
- added joint arm_joint: type fixed, parent base_link, child arm_base_link, origin xyz=1 -1 0.0 rpy=0.0 0.0 0.524
